File: hardware/ComponentTester/ComponentTester.kicad_pcb (KiCad board)
At the start: 2 copper layers, 51 x 90.6 mm, 18 parts, among them J1 Conn_01x06_Socket, J2 AVR-ISP-6, J3 Conn_02x07_Counter_Clockwise, J4 GameBoy_GamePak_DMG-09, J5 Conn_01x03_Pin, SW1 SW_Push, U1 ATmega328P-A

Commit message: hardware changes
Parts:
- U1: value ATmega328P-A -> ATmega328PB-A
- moved J2 45.6 mm to (89.0, 89.6)
- turned C2 to 180 degrees
Connections:
- U1 pad 19: /CARD_A0 -> /CARD_A2
- U1 pad 22: /CARD_A1 -> /CARD_A3
- U1 pad 3: GND -> /CARD_A0
- U1 pad 6: +5V -> /CARD_A1
Routing:
- net /CARD_~{RES}: track 32.1 -> 74.4 mm, vias 1 -> 4
- net /CARD_A3: track 0.00 -> 37.9 mm, vias 0 -> 2
- net /CARD_A2: track 0.00 -> 32.2 mm, vias 0 -> 2
- net /CARD_D5: track 43.8 -> 67.9 mm, vias 4 -> 2
- net +5V: track 135.3 -> 158.9 mm
- net /CARD_D4: track 40.6 -> 62.7 mm, vias 3 -> 2
- net GND: track 21.0 -> 5.95 mm, vias 140 -> 129
- net /CARD_D3: track 49.1 -> 57.1 mm, vias 3 -> 2
- net /CARD_CLK: track 110.7 -> 117.5 mm
- net /CARD_A0: track 38.0 -> 42.1 mm
- net /2: track 95.3 -> 92.2 mm
- net /CARD_A15: track 55.7 -> 58.4 mm
- net /CARD_A1: track 40.2 -> 38.4 mm
- net Net-(U1-PD5): track 14.1 -> 12.6 mm
- net /CARD_~{WR}: track 48.4 -> 50.0 mm
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Other:
- outline, holes or cut-outs redrawn
- board text added: "Component-Tester V1.1"
- board text removed: "Component-Tester V1.0"
