File: hardware/ComponentTester/ComponentTester.kicad_sch (KiCad schematic)
At the start: 17 parts, among them J1 Conn_01x06_Socket, J2 AVR-ISP-6, J3 Conn_02x07_Counter_Clockwise, J4 GameBoy_GamePak_DMG-09, SW1 SW_Push, U1 ATmega328P-A

Commit message: some work
Parts:
- added J5: Conn_01x03_Pin, MyLibrary:Component_Testpad, symbol Connector:Conn_01x03_Pin
Connections:
- net +5V: now also C2.1, U1.4 (VCC), U1.6 (VCC)
- net 1: now also J3.10 (Pin_10), J3.11 (Pin_11), J3.14 (Pin_14), J3.8 (Pin_8), J3.9 (Pin_9), J5.3 (Pin_3); no longer J3.1 (Pin_1), J3.2 (Pin_2), J3.3 (Pin_3), J3.4 (Pin_4), J3.7 (Pin_7)
- net 2: now also J3.1 (Pin_1), J3.13 (Pin_13), J3.2 (Pin_2), J3.3 (Pin_3), J5.2 (Pin_2); no longer J3.10 (Pin_10), J3.6 (Pin_6), J3.8 (Pin_8), J3.9 (Pin_9)
- net 3: now also J3.4 (Pin_4), J3.6 (Pin_6), J3.7 (Pin_7), J5.1 (Pin_1); no longer J3.11 (Pin_11), J3.13 (Pin_13), J3.14 (Pin_14)
Other:
- note added: "Flash and program: https://wolles-elektronikkiste.de/atmega328p-standalone-betreiben"
- note removed: "Flash and program: https://electronoobs.com/eng_arduino_tut33.php https://wolles-elektronikkiste.de/atmega328p-standalone-betreiben"
- moved on the sheet: J3
Changed lines of the file:
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@@
 	(generator_version "9.0")
 	(paper "A4")
-	(text "Flash and program:\nhttps://electronoobs.com/eng_arduino_tut33.php\nhttps://wolles-elektronikkiste.de/atmega328p-standalone-betreiben"
+	(text "Flash and program:\nhttps://wolles-elektronikkiste.de/atmega328p-standalone-betreiben"
 		(exclude_from_sim no)
 		(at 54.356 166.624 0)
@@
 	)
 	(junction
+		(at 76.2 72.39)
+		(diameter 0)
+		(color 0 0 0 0)
+	)
+	(junction
 		(at 101.6 91.44)
 		(diameter 0)
@@
 	)
 	(junction
+		(at 73.66 72.39)
+		(diameter 0)
+		(color 0 0 0 0)
+	)
+	(junction
 		(at 93.98 111.76)
 		(diameter 0)
@@
 	(wire
 		(pts
-			(xy 175.26 97.79) (xy 175.26 100.33)
-		)
-		(stroke
-			(width 0)
-			(type default)
-		)
-	)
-	(wire
-		(pts
 			(xy 180.34 97.79) (xy 180.34 100.33)
 		)
@@
 	(wire
 		(pts
+			(xy 170.18 91.44) (xy 170.18 100.33)
+		)
+		(stroke
+			(width 0)
+			(type default)
+		)
+	)
+	(wire
+		(pts
 			(xy 116.84 121.92) (xy 116.84 119.38)
 		)
@@
 	(wire
 		(pts
+			(xy 172.72 91.44) (xy 172.72 100.33)
+		)
+		(stroke
+			(width 0)
+			(type default)
+		)
+	)
+	(wire
+		(pts
 			(xy 106.68 96.52) (xy 88.9 96.52)
 		)
@@
 	(wire
 		(pts
-			(xy 170.18 97.79) (xy 170.18 100.33)
-		)
-		(stroke
-			(width 0)
-			(type default)
-		)
-	)
-	(wire
-		(pts
 			(xy 57.15 81.28) (xy 58.42 81.28)
 		)
@@
 	(wire
 		(pts
-			(xy 172.72 97.79) (xy 172.72 100.33)
-		)
-		(stroke
-			(width 0)
-			(type default)
-		)
-	)
-	(wire
-		(pts
 			(xy 88.9 91.44) (xy 101.6 91.44)
 		)
@@
 	(wire
 		(pts
-			(xy 76.2 66.04) (xy 76.2 73.66)
+			(xy 76.2 66.04) (xy 76.2 72.39)
 		)
 		(stroke
@@
 	(wire
 		(pts
+			(xy 73.66 72.39) (xy 76.2 72.39)
+		)
+		(stroke
+			(width 0)
+			(type default)
+		)
+	)
+	(wire
+		(pts
+			(xy 175.26 91.44) (xy 175.26 100.33)
+		)
+		(stroke
+			(width 0)
+			(type default)
+		)
+	)
+	(wire
+		(pts
 			(xy 143.51 125.73) (xy 143.51 127)
 		)
@@
 	(wire
 		(pts
+			(xy 76.2 72.39) (xy 76.2 73.66)
+		)
+		(stroke
+			(width 0)
+			(type default)
+		)
+	)
+	(wire
+		(pts
 			(xy 99.06 88.9) (xy 88.9 88.9)
 		)
@@
 		)
 	)
+	(label "MISO"
+		(at 90.17 91.44 0)
+		(effects
+			(font
+				(size 1.27 1.27)
+			)
+			(justify left bottom)
+		)
+	)
 	(label "ADC1"
 		(at 90.17 106.68 0)
@@
 		)
 	)
+	(label "SCK"
+		(at 90.17 93.98 0)
+		(effects
+			(font
+				(size 1.27 1.27)
+			)
+			(justify left bottom)
+		)
+	)
 	(label "CARD_~{WR}"
 		(at 101.6 156.21 90)
@@
 		)
 	)
+	(label "MOSI"
+		(at 90.17 88.9 0)
+		(effects
+			(font
+				(size 1.27 1.27)
+			)
+			(justify left bottom)
+		)
+	)
 	(label "CARD_D3"
 		(at 99.06 59.69 270)
@@
 	)
 	(symbol
+		(lib_id "Connector:Conn_01x03_Pin")
+		(at 172.72 86.36 270)
+		(unit 1)
+		(exclude_from_sim no)
+		(in_bom yes)
+		(on_board yes)
+		(dnp no)
+		(property "Reference" "J5"
+			(at 172.72 81.28 90)
+			(effects
+				(font
+					(size 1.27 1.27)
+				)
+			)
+		)
+		(property "Value" "Conn_01x03_Pin"
+			(at 172.72 83.82 90)
+			(effects
+				(font
+					(size 1.27 1.27)
+				)
+			)
+		)
+		(property "Footprint" "MyLibrary:Component_Testpad"
+			(at 172.72 86.36 0)
+			(effects
+				(font
+					(size 1.27 1.27)
+				)
+				(hide yes)
+			)
+		)
+		(property "Datasheet" "~"
+			(at 172.72 86.36 0)
+			(effects
+				(font
+					(size 1.27 1.27)
+				)
+				(hide yes)
+			)
+		)
+		(property "Description" "Generic connector, single row, 01x03, script generated"
+			(at 172.72 86.36 0)
+			(effects
+				(font
+					(size 1.27 1.27)
+				)
+				(hide yes)
+			)
+		)
+		(pin "3"
+		)
+		(pin "2"
+		)
+		(pin "1"
+		)
+		(instances
+			(project ""
+				(path "/80bd7774-bbdd-4a53-bd07-874de5be49cb"
+					(reference "J5")
+					(unit 1)
+				)
+			)
+		)
+	)
+	(symbol
 		(lib_id "Device:R")
 		(at 120.65 115.57 0)
@@
 	(symbol
 		(lib_id "Connector_Generic:Conn_02x07_Counter_Clockwise")
-		(at 177.8 105.41 270)
+		(at 177.8 107.95 90)
 		(unit 1)
 		(exclude_from_sim no)
@@
 		(dnp no)
 		(property "Reference" "J3"
-			(at 167.132 105.664 90)
+			(at 188.468 107.696 90)
 			(effects
 				(font
@@
 		)
 		(property "Value" "Conn_02x07_Counter_Clockwise"
-			(at 183.642 117.348 90)
+			(at 179.324 117.602 90)
 			(effects
 				(font
@@
 		)
 		(property "Footprint" "Socket:DIP_Socket-14_W4.3mm_W5.08mm_W7.62mm_W10.16mm_W10.9mm_3M_214-3339-00-0602J"
-			(at 177.8 105.41 0)
+			(at 177.8 107.95 0)
 			(effects
 				(font
@@
 		)
 		(property "Datasheet" "~"
-			(at 177.8 105.41 0)
+			(at 177.8 107.95 0)
 			(effects
 				(font
@@
 		)
 		(property "Description" "Generic connector, double row, 02x07, counter clockwise pin numbering scheme (similar to DIP package numbering), script generated (kicad-library-utils/schlib/autogen/connector/)"
-			(at 177.8 105.41 0)
+			(at 177.8 107.95 0)
 			(effects
 				(font

Commit message: hardware changes
Parts:
- removed U1: ATmega328P-A, Package_QFP:TQFP-32_7x7mm_P0.8mm, symbol MCU_Microchip_ATmega:ATmega328P-A
- added U1: ATmega328PB-A, Package_QFP:TQFP-32_7x7mm_P0.8mm, symbol MCU_Microchip_ATmega:ATmega328PB-A
Connections:
- net +5V: now also U1.18 (AVCC), U1.4 (VCC)
- net 1: now also U1.23 (PC0)
- net 2: now also U1.24 (PC1)
- net 3: now also U1.25 (PC2)
- net CARD_A0: now also U1.3 (PE0)
- net CARD_A1: now also U1.6 (PE1)
- net CARD_A15: now also U1.31 (PD1)
- net CARD_A2: now also U1.19 (PE2)
- net CARD_A3: now also U1.22 (PE3)
- net CARD_CLK: now also U1.26 (PC3)
- net CARD_D0: now also U1.12 (PB0)
- net CARD_D1: now also U1.13 (PB1)
- net CARD_D2: now also U1.14 (PB2)
- net CARD_D3: now also U1.15 (PB3)
- net CARD_D4: now also U1.16 (PB4)
- net CARD_D5: now also U1.17 (PB5)
- net CARD_D6: now also U1.7 (XTAL1/PB6)
- net CARD_D7: now also U1.8 (XTAL2/PB7)
- net CARD_~{CS}: now also U1.30 (PD0)
- net CARD_~{RD}: now also U1.28 (PC5)
- net CARD_~{RES}: now also U1.29 (~{RESET}/PC6)
- net CARD_~{WR}: now also U1.27 (PC4)
- net GND: now also U1.21 (GND), U1.5 (GND)
- net at R1.2: now also U1.32 (PD2)
- net at C1.1: now also U1.20 (AREF)
- net at R3.2: now also U1.2 (PD4)
- net at R4.2: now also U1.9 (PD5)
- net at R2.2: now also U1.1 (PD3)
- net at R5.2: now also U1.10 (PD6)
- net at R6.2: now also U1.11 (PD7)
- no-connect marks 14 -> 12
Other:
- note added: "D0-D7: data A0-A3: data WR|RD|CS|VIN: control CLK: button RES: reset <-> pull low VIN-A15: indicator"
- note removed: "D0-D7: data ADC6,ADC7: data WR|RD|CS|VIN: control CLK: button RES: reset <-> pull low VIN-A15: indicator"
Changed lines of the file:
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@@
 		)
 	)
-	(text "D0-D7: data\nADC6,ADC7: data\nWR|RD|CS|VIN: control\nCLK: button\nRES: reset <-> pull low\nVIN-A15: indicator"
+	(text "D0-D7: data\nA0-A3: data\nWR|RD|CS|VIN: control\nCLK: button\nRES: reset <-> pull low\nVIN-A15: indicator"
 		(exclude_from_sim no)
 		(at 209.296 48.006 0)
@@
 	)
 	(no_connect
-		(at 209.55 85.09)
-	)
-	(no_connect
 		(at 209.55 115.57)
 	)
@@
 	)
 	(no_connect
-		(at 209.55 87.63)
-	)
-	(no_connect
 		(at 209.55 97.79)
 	)
@@
 	(wire
 		(pts
+			(xy 49.53 132.08) (xy 58.42 132.08)
+		)
+		(stroke
+			(width 0)
+			(type default)
+		)
+	)
+	(wire
+		(pts
 			(xy 109.22 99.06) (xy 88.9 99.06)
 		)
@@
 	(wire
 		(pts
-			(xy 49.53 86.36) (xy 58.42 86.36)
+			(xy 49.53 124.46) (xy 58.42 124.46)
 		)
 		(stroke
@@
 	(wire
 		(pts
-			(xy 49.53 88.9) (xy 58.42 88.9)
+			(xy 49.53 127) (xy 58.42 127)
 		)
 		(stroke
@@
 	(wire
 		(pts
+			(xy 49.53 129.54) (xy 58.42 129.54)
+		)
+		(stroke
+			(width 0)
+			(type default)
+		)
+	)
+	(wire
+		(pts
 			(xy 143.51 125.73) (xy 143.51 127)
 		)
@@
 	)
 	(label "CARD_A0"
-		(at 49.53 86.36 0)
+		(at 49.53 124.46 0)
 		(effects
 			(font
@@
 		)
 	)
+	(label "CARD_A2"
+		(at 49.53 129.54 0)
+		(effects
+			(font
+				(size 1.27 1.27)
+			)
+			(justify left bottom)
+		)
+	)
 	(label "CARD_CLK"
 		(at 93.98 156.21 90)
@@
 	)
 	(label "CARD_A1"
-		(at 49.53 88.9 0)
+		(at 49.53 127 0)
 		(effects
 			(font
@@
 		)
 	)
+	(label "CARD_A3"
+		(at 49.53 132.08 0)
+		(effects
+			(font
+				(size 1.27 1.27)
+			)
+			(justify left bottom)
+		)
+	)
 	(label "3"
 		(at 182.88 115.57 180)
@@
 	)
 	(symbol
-		(lib_id "MCU_Microchip_ATmega:ATmega328P-A")
-		(at 73.66 111.76 0)
-		(unit 1)
-		(exclude_from_sim no)
-		(in_bom yes)
-		(on_board yes)
-		(dnp no)
-		(property "Reference" "U1"
-			(at 79.248 73.914 0)
-			(effects
-				(font
-					(size 1.27 1.27)
-				)
-				(justify left)
-			)
-		)
-		(property "Value" "ATmega328P-A"
-			(at 72.136 113.03 90)
-			(effects
-				(font
-					(size 1.27 1.27)
-				)
-				(justify left)
-			)
-		)
-		(property "Footprint" "Package_QFP:TQFP-32_7x7mm_P0.8mm"
-			(at 73.66 111.76 0)
-			(effects
-				(font
-					(size 1.27 1.27)
-					(italic yes)
-				)
-				(hide yes)
-			)
-		)
-		(property "Datasheet" "https://ww1.microchip.com/downloads/aemDocuments/documents/MCU08/ProductDocuments/DataSheets/ATmega48A-PA-88A-PA-168A-PA-328-P-DS-DS40002061B.pdf"
-			(at 73.66 111.76 0)
-			(effects
-				(font
-					(size 1.27 1.27)
-				)
-				(hide yes)
-			)
-		)
-		(property "Description" "20MHz, 32kB Flash, 2kB SRAM, 1kB EEPROM, TQFP-32"
-			(at 73.66 111.76 0)
-			(effects
-				(font
-					(size 1.27 1.27)
-				)
-				(hide yes)
-			)
-		)
-		(pin "10"
-		)
-		(pin "30"
-		)
-		(pin "13"
-		)
-		(pin "32"
-		)
-		(pin "22"
-		)
-		(pin "23"
-		)
-		(pin "27"
-		)
-		(pin "28"
-		)
-		(pin "6"
-		)
-		(pin "29"
-		)
-		(pin "19"
-		)
-		(pin "4"
-		)
-		(pin "31"
-		)
-		(pin "21"
-		)
-		(pin "3"
-		)
-		(pin "18"
-		)
-		(pin "20"
-		)
-		(pin "26"
-		)
-		(pin "2"
-		)
-		(pin "1"
-		)
-		(pin "17"
-		)
-		(pin "25"
-		)
-		(pin "14"
-		)
-		(pin "24"
-		)
-		(pin "11"
-		)
-		(pin "12"
-		)
-		(pin "16"
-		)
-		(pin "9"
-		)
-		(pin "5"
-		)
-		(pin "8"
-		)
-		(pin "15"
-		)
-		(pin "7"
-		)
-		(instances
-			(project ""
-				(path "/80bd7774-bbdd-4a53-bd07-874de5be49cb"
-					(reference "U1")
-					(unit 1)
-				)
-			)
-		)
-	)
-	(symbol
 		(lib_id "Connector:Conn_01x06_Socket")
 		(at 158.75 129.54 0)
@@
 					(unit 1)
 				)
+			)
+		)
+	)
+	(symbol
+		(lib_id "MCU_Microchip_ATmega:ATmega328PB-A")
+		(at 73.66 111.76 0)
+		(unit 1)
+		(exclude_from_sim no)
+		(in_bom yes)
+		(on_board yes)
+		(dnp no)
+		(property "Reference" "U1"
+			(at 83.058 74.422 0)
+			(effects
+				(font
+					(size 1.27 1.27)
+				)
+				(justify left)
+			)
+		)
+		(property "Value" "ATmega328PB-A"
+			(at 73.406 120.396 90)
+			(effects
+				(font
+					(size 1.27 1.27)
+				)
+				(justify left)
+			)
+		)
+		(property "Footprint" "Package_QFP:TQFP-32_7x7mm_P0.8mm"
+			(at 73.66 111.76 0)
+			(effects
+				(font
+					(size 1.27 1.27)
+					(italic yes)
+				)
+				(hide yes)
+			)
+		)
+		(property "Datasheet" "http://ww1.microchip.com/downloads/en/DeviceDoc/40001906C.pdf"
+			(at 73.66 111.76 0)
+			(effects
+				(font
+					(size 1.27 1.27)
+				)
+				(hide yes)
+			)
+		)
+		(property "Description" "20MHz, 32kB Flash, 2kB SRAM, 1kB EEPROM, TQFP-32"
+			(at 73.66 111.76 0)
+			(effects
+				(font
+					(size 1.27 1.27)
+				)
+				(hide yes)
+			)
+		)
+		(pin "11"
+		)
+		(pin "12"
+		)
+		(pin "23"
+		)
+		(pin "22"
+		)
+		(pin "16"
+		)
+		(pin "4"
+		)
+		(pin "21"
+		)
+		(pin "7"
+		)
+		(pin "25"
+		)
+		(pin "31"
+		)
+		(pin "15"
+		)
+		(pin "29"
+		)
+		(pin "14"
+		)
+		(pin "1"
+		)
+		(pin "2"
+		)
+		(pin "20"
+		)
+		(pin "9"
+		)
+		(pin "10"
+		)
+		(pin "13"
+		)
+		(pin "3"
+		)
+		(pin "26"
+		)
+		(pin "27"
+		)
+		(pin "17"
+		)
+		(pin "28"
+		)
+		(pin "8"
+		)
+		(pin "19"
+		)
+		(pin "30"
+		)
+		(pin "18"
+		)
+		(pin "6"
+		)
+		(pin "24"
+		)
+		(pin "5"
+		)
+		(pin "32"
+		)
+		(instances
+			(project ""
+				(path "/80bd7774-bbdd-4a53-bd07-874de5be49cb"
+					(reference "U1")
+					(unit 1)
+				)
